File: hardware/rev-a/pendant-rev-a.kicad_sch (KiCad schematic)
At the start: 84 parts, among them J1 USB-C USB2 receptacle TBD, J2 Protected 1S 100mAh pack + NTC, J3 SWD pads, Q1 P-MOS low Vth TBD, Q2 2N7002 (charge inhibit), Q3 2N7002 (VBUS detect), SW1 REC button, U1 STM32U535RCT6, U10 TPS22916CYFPR, U11 CSNP32GCR01-BOW, U2 USBLC6-2SC6, U3 BQ25101YFPR, U4 TPS7A0230PDBVR, U5 TPS7A0233PDBVR, U6 TPS7A0218PDBVR, U7 MAX17048G+T10, U8 T5838, U9 TXS0104EYZTR, Y1 32.768kHz CL=7pF TBD

Commit message: Require on-device indicators and add battery and status LED circuits
Parts:
- added D3: amber LED 0402 TBD, symbol Pendant:Part_D3
- added D4: amber LED 0402 TBD, symbol Pendant:Part_D4
- added D5: amber LED 0402 TBD, symbol Pendant:Part_D5
- added D6: amber LED 0402 TBD, symbol Pendant:Part_D6
- added R29: 6.8k tentative, symbol Pendant:Part_R29
- added R30: 6.8k tentative, symbol Pendant:Part_R30
- added R31: 6.8k tentative, symbol Pendant:Part_R31
- added R32: 6.8k tentative, symbol Pendant:Part_R32
Connections:
- net GND: now also D3.2 (K), D4.2 (K), D5.2 (K), D6.2 (K)
- net BAT_LED_1: now reaches U1.20 (PA4)
- net BAT_LED_1: now also R29.1
- net BAT_LED_2: now reaches U1.21 (PA5)
- net BAT_LED_2: now also R30.1
- net BAT_LED_3: now reaches U1.22 (PA6)
- net BAT_LED_3: now also R31.1
- net STATUS_LED: now reaches U1.23 (PA7)
- net STATUS_LED: now also R32.1
- new net BAT_LED_1_A: D3.1 (A), R29.2
- new net BAT_LED_2_A: D4.1 (A), R30.2
- new net BAT_LED_3_A: D5.1 (A), R31.2
- new net STATUS_LED_A: D6.1 (A), R32.2
- no-connect marks 29 -> 25
Other:
- note added: "04 AUDIO / SD / INDICATORS"
- note removed: "04 OMI AUDIO / SD NAND"

Commit message: Add A1 netted PCB placement study and package footprints
Parts:
- C1, C10, C11, C12, C13, C14, C16, C17, C18, C19, C2, C20, C21, C22, C23, C24, C25, C26, C3, C6, C7, C8, C9: footprint (none) -> Capacitor_SMD:C_0402_1005Metric
- C15, C27, C4, C5: footprint (none) -> Capacitor_SMD:C_0603_1608Metric
- D1, D3, D4, D5, D6: footprint (none) -> LED_SMD:LED_0402_1005Metric
- D2: value Schottky 20V >=200mA TBD -> BAT54WS (candidate; leakage/forward drop review pending); footprint (none) -> Diode_SMD:D_SOD-323
- J1: value USB-C USB2 receptacle TBD -> USB4105-GF-A (candidate); footprint (none) -> Connector_USB:USB_C_Receptacle_GCT_USB4105-xx-A_16P_TopMnt_Horizontal
- J2: value Protected 1S 100mAh pack + NTC -> S2B-PH-SM4-TB(LF)(SN) / DTP401525 110mAh; footprint (none) -> Connector_JST:JST_PH_S2B-PH-SM4-TB_1x02-1MP_P2.00mm_Horizontal
- J3: footprint (none) -> Pendant:SWD_5Pad_Pogo
- Q1: value P-MOS low Vth TBD -> DMP2035U (candidate; power path review pending); footprint (none) -> Package_TO_SOT_SMD:SOT-23
- Q2, Q3: footprint (none) -> Package_TO_SOT_SMD:SOT-23
- R1, R11, R12, R13, R14, R15, R16, R17, R18, R19, R2, R20, R21, R22, R23, R24, R25, R26, R27, R28, R29, R3, R30, R31, R32, R4, R5, R6, R7, R8, R9, TH1: footprint (none) -> Resistor_SMD:R_0402_1005Metric
- R10: value 2.7k 1% -> 6.19k 1%; footprint (none) -> Resistor_SMD:R_0402_1005Metric
- SW1: value REC button -> B3U-1000P (candidate); footprint (none) -> Button_Switch_SMD:SW_SPST_B3U-1000P
- TP1, TP2, TP3, TP4, TP5, TP6, TP7: footprint (none) -> TestPoint:TestPoint_Pad_D1.0mm
- U10: footprint (none) -> Pendant:TPS22916_YFP4
- U11: footprint (none) -> Pendant:CSNP32GCR01_LGA8
- U2: footprint (none) -> Package_TO_SOT_SMD:SOT-23-6
- U3: footprint (none) -> Pendant:BQ25101_YFP6
- U4, U5, U6: footprint (none) -> Package_TO_SOT_SMD:SOT-23-5
- U7: footprint (none) -> Package_DFN_QFN:TDFN-8-1EP_2x2mm_P0.5mm_EP0.8x1.2mm
- U8: footprint (none) -> Pendant:T5838_LGA7_BottomPort
- U9: footprint (none) -> Pendant:TXS0104E_YZT12
- Y1: footprint (none) -> Crystal:Crystal_SMD_2012-2Pin_2.0x1.2mm
Connections:
- net BAT_LED_1_A: now also D3.2 (A); no longer D3.1 (A)
- net BAT_LED_2_A: now also D4.2 (A); no longer D4.1 (A)
- net BAT_LED_3_A: now also D5.2 (A); no longer D5.1 (A)
- net BAT_TS: no longer J2.3 (NTC)
- net GND: now also D1.1 (K), D3.1 (K), D4.1 (K), D5.1 (K), D6.1 (K), J1.SH (SHIELD); no longer D1.2 (K), D3.2 (K), D4.2 (K), D5.2 (K), D6.2 (K), J1.S1 (SHIELD)
- net LED_A: now also D1.2 (A); no longer D1.1 (A)
- net STATUS_LED_A: now also D6.2 (A); no longer D6.1 (A)
- net SYS: now also D2.1 (K); no longer D2.2 (K)
- net VBUS: now also D2.2 (A); no longer D2.1 (A)
Other:
- note added: "A1 ENGINEERING DRAFT - NOT FOR FABRICATION - See hardware/rev-a/README.md"
- note removed: "A0 ENGINEERING DRAFT - NOT FOR FABRICATION - See hardware/rev-a/README.md"
- moved on the sheet: Q2, Q3, R12, R13, R14, R15, TH1
Changed lines of the file:
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@@
 (kicad_sch (version 20250114) (generator "eeschema") (paper "A0")
- (title_block (title "Pendant Recorder - Omi-derived electrical design") (date "2026-10-24") (rev "A0 DRAFT") (comment 1 "No PCB / no manufacturing release"))
+ (title_block (title "Pendant Recorder - Omi-derived electrical design") (date "2026-10-24") (rev "A1 DRAFT") (comment 1 "Unrouted PCB / no manufacturing release"))

Commit message: Advance v1 sourcing audit, standard SWD connection and audio profile validation
Parts:
- J3: value SWD pads -> TC2030-CTX-NL-STDC14 target pads; footprint Pendant:SWD_5Pad_Pogo -> Connector:Tag-Connect_TC2030-IDC-NL_2x03_P1.27mm_Vertical
Connections:
- net GND: now also J3.5 (GND); no longer J3.3 (GND)
- net NRST: now also J3.3 (nRESET); no longer J3.5 (NRST)
- no-connect marks 25 -> 26
