File: hardware/omi-fit-d1/omi-fit-d1.kicad_sch (KiCad schematic)
At the start: 76 parts, among them J1 USB4105-GF-A (candidate), J2 SM02B-SRSS-TB / factory prote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, J3 TC2030 SWD target pads, Q1 DMP2035U (candidate; power pa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, Q2 2N7002 (charge inhibit), Q3 2N7002 (VBUS detect), SW1 B3U-1000P (candidate), U1 STM32U535CEU6, U10 TPS22916CYFPR, U11 CSNP32GCR01-BOW, U2 USBLC6-2P6, U3 BQ25101YFPR, U4 TPS7A0233PDBVR, U6 TPS7A0218PDBVR, U8 T5838, U9 TXS0104ERUTR, Y1 32.768kHz CL=7pF TBD

Commit message: Route circular D1.1 and prepare unreleased DFM package
Parts:
- J1: footprint Connector_USB:USB_C_Receptacle_GCT_USB4105-xx-A_16P_TopMnt_Horizontal -> PendantD1:USB_C_GCT_USB4105_GroundLand112
Connections:
- net MIC_EN: now also U1.41 (PB5); no longer U1.19 (PB1)
